File: hardware/multiboard_controller/Input Connectors.kicad_sch (KiCad schematic)
At the start: 10 parts, among them J1 USB_C_Receptacle, U4 MAX38908xTD

Commit message: Add Channel Select switches and USB output ports
Connections:
- net D+ renamed host_USB_D_P
- net D- renamed host_USB_D_N
Other:
- title: (none) -> Input Connectors
Changed lines of the file:
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@@
 	(generator_version "8.0")
 	(paper "A4")
+	(title_block
+		(title "Input Connectors")
+		(date "2025-02-11")
+	)
 	(junction
 		(at 241.3 86.36)
@@
 		)
 	)
-	(global_label "D-"
+	(global_label "host_USB_D_P"
+		(shape input)
+		(at 127 78.74 0)
+		(fields_autoplaced yes)
+		(effects
+			(font
+				(size 1.27 1.27)
+			)
+			(justify left)
+		)
+		(property "Intersheetrefs" "${INTERSHEET_REFS}"
+			(at 142.7179 78.6606 0)
+			(effects
+				(font
+					(size 1.27 1.27)
+				)
+				(justify left)
+				(hide yes)
+			)
+		)
+	)
+	(global_label "host_USB_D_N"
 		(shape input)
 		(at 127 73.66 0)
@@
 		)
 		(property "Intersheetrefs" "${INTERSHEET_REFS}"
-			(at 132.8276 73.66 0)
+			(at 142.7783 73.5806 0)
 			(effects
 				(font
-					(size 1.27 1.27)
-				)
-				(justify left)
-				(hide yes)
-			)
-		)
-	)
-	(global_label "D+"
-		(shape input)
-		(at 127 78.74 0)
-		(fields_autoplaced yes)
-		(effects
-			(font
-				(size 1.27 1.27)
-			)
-			(justify left)
-		)
-		(property "Intersheetrefs" "${INTERSHEET_REFS}"
-			(at 132.8276 78.74 0)
-			(effects
-				(font

Commit message: Connecting first UART line out from mux
Connections:
- net V_BUS: now reaches C2.2, J1.A4 (VBUS), J1.A9 (VBUS), J1.B4 (VBUS), J1.B9 (VBUS), U4.1 (IN), U4.2 (IN), U4.3 (IN), U4.4 (IN)
Changed lines of the file:
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@@
+		)
+	)
+	(global_label "V_BUS"
+		(shape input)
+		(at 151.13 58.42 90)
+		(fields_autoplaced yes)
+		(effects
+			(font
+				(size 1.27 1.27)
+			)
+			(justify left)
+		)
+		(property "Intersheetrefs" "${INTERSHEET_REFS}"
+			(at 151.13 49.5686 90)
+			(effects
+				(font
+					(size 1.27 1.27)
+				)
+				(justify left)
+				(hide yes)
+			)
 		)
 	)

Commit message: Starting layout
Add serial ground connections, add footprint libraries, start layout.
Parts:
- J1: footprint (none) -> Connector_USB:USB_C_Receptacle_GCT_USB4135-GF-A_6P_TopMnt_Horizontal
- R3, R4: footprint (none) -> Resistor_SMD:R_0402_1005Metric
Changed lines of the file:
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@@
 			)
 		)
-		(property "Footprint" ""
+		(property "Footprint" "Connector_USB:USB_C_Receptacle_GCT_USB4135-GF-A_6P_TopMnt_Horizontal"
 			(at 105.41 83.82 0)
 			(effects
@@
 			)
 		)
-		(property "Footprint" ""
+		(property "Footprint" "Resistor_SMD:R_0402_1005Metric"
 			(at 124.714 62.484 90)
 			(effects
@@
 			)
 		)
-		(property "Footprint" ""
+		(property "Footprint" "Resistor_SMD:R_0402_1005Metric"
 			(at 124.714 65.024 90)
 			(effects
