File: hardware/multiboard_controller/multiboard_controller.kicad_pcb (KiCad board)
At the start: 2 copper layers, 1 part, among them U4 MAX38908xTD

Commit message: Starting layout
Add serial ground connections, add footprint libraries, start layout.
Parts:
- added C1: 22uF, all-footprints:G-188_MUR, F.Cu at (321.5, 110.2)
- added C2: 22uF, all-footprints:G-188_MUR, F.Cu at (333.7, 111.5)
- added C3: 47nF, all-footprints:CAPC10555_55N_KEM, F.Cu at (324.6, 112.5)
- added C4: 1uF, all-footprints:CAP_CL05_SAM, F.Cu at (333.8, 110.0)
- added C5: 18pF, Capacitor_SMD:C_0402_1005Metric, F.Cu at (226.0, 213.0)
- added C6: 18pF, Capacitor_SMD:C_0402_1005Metric, F.Cu at (228.0, 213.0)
- added D1: TXLED, LED_SMD:LED_0805_2012Metric, F.Cu at (238.9, 200.5)
- added D2: RXLED, LED_SMD:LED_0805_2012Metric, F.Cu at (238.9, 203.0)
- added J1: USB_C_Receptacle, Connector_USB:USB_C_Receptacle_GCT_USB4135-GF-A_6P_TopMnt_Horizontal, F.Cu at (302.5, 186.0)
- added J10: DE9_Plug_MountingHoles, all-footprints:ASSMANN_A-DS_09_A_KG-T2S, F.Cu at (366.0, 332.5)
- added J11: DE9_Plug_MountingHoles, all-footprints:ASSMANN_A-DS_09_A_KG-T2S, F.Cu at (331.5, 332.5)
- added J12: DE9_Plug_MountingHoles, all-footprints:ASSMANN_A-DS_09_A_KG-T2S, F.Cu at (297.0, 332.5)
- added J13: DE9_Plug_MountingHoles, all-footprints:ASSMANN_A-DS_09_A_KG-T2S, F.Cu at (263.0, 332.5)
- added J15: DE9_Plug_MountingHoles, all-footprints:ASSMANN_A-DS_09_A_KG-T2S, F.Cu at (229.0, 332.5)
- added J16: DE9_Plug_MountingHoles, all-footprints:ASSMANN_A-DS_09_A_KG-T2S, F.Cu at (195.1, 332.6)
- added J17: DE9_Plug_MountingHoles, all-footprints:ASSMANN_A-DS_09_A_KG-T2S, F.Cu at (161.4, 332.5)
- added J18: DE9_Plug_MountingHoles, all-footprints:ASSMANN_A-DS_09_A_KG-T2S, F.Cu at (127.5, 332.5)
- added J2: USB_C_Receptacle, Connector_USB:USB_C_Receptacle_GCT_USB4135-GF-A_6P_TopMnt_Horizontal, F.Cu at (-50.2, -64.7)
- added J3: USB_C_Receptacle, Connector_USB:USB_C_Receptacle_GCT_USB4135-GF-A_6P_TopMnt_Horizontal, F.Cu at (-50.2, -55.5)
- added J4: USB_C_Receptacle, Connector_USB:USB_C_Receptacle_GCT_USB4135-GF-A_6P_TopMnt_Horizontal, F.Cu at (-50.2, -46.2)
- added J5: USB_C_Receptacle, Connector_USB:USB_C_Receptacle_GCT_USB4135-GF-A_6P_TopMnt_Horizontal, F.Cu at (-50.2, -37.0)
- added J6: USB_C_Receptacle, Connector_USB:USB_C_Receptacle_GCT_USB4135-GF-A_6P_TopMnt_Horizontal, F.Cu at (-50.2, -27.7)
- added J7: USB_C_Receptacle, Connector_USB:USB_C_Receptacle_GCT_USB4135-GF-A_6P_TopMnt_Horizontal, F.Cu at (-50.2, -18.5)
- added J8: USB_C_Receptacle, Connector_USB:USB_C_Receptacle_GCT_USB4135-GF-A_6P_TopMnt_Horizontal, F.Cu at (-50.2, -9.22)
- added J9: USB_C_Receptacle, Connector_USB:USB_C_Receptacle_GCT_USB4135-GF-A_6P_TopMnt_Horizontal, F.Cu at (-21.5, -1.50)
- added R1: 15K, all-footprints:RC0402N_PAN, F.Cu at (324.6, 109.5)
- added R10: 5.1K, Resistor_SMD:R_0402_1005Metric, F.Cu at (-38.8, -66.5)
- added R11: 5.1K, Resistor_SMD:R_0402_1005Metric, F.Cu at (-38.8, -64.5)
- added R12: 5.1K, Resistor_SMD:R_0402_1005Metric, F.Cu at (-38.8, -62.5)
- added R13: 5.1K, Resistor_SMD:R_0402_1005Metric, F.Cu at (-35.9, -68.4)
- added R14: 5.1K, Resistor_SMD:R_0402_1005Metric, F.Cu at (-35.9, -66.5)
- added R15: 5.1K, Resistor_SMD:R_0402_1005Metric, F.Cu at (-35.9, -64.5)
- added R16: 5.1K, Resistor_SMD:R_0402_1005Metric, F.Cu at (-35.9, -62.5)
- added R17: 5.1K, Resistor_SMD:R_0402_1005Metric, F.Cu at (-33.0, -68.5)
- added R18: 5.1K, Resistor_SMD:R_0402_1005Metric, F.Cu at (-33.0, -66.5)
- added R19: 5.1K, Resistor_SMD:R_0402_1005Metric, F.Cu at (-33.0, -64.5)
- added R2: 68.1K, all-footprints:RC0402N_PAN, F.Cu at (324.5, 111.0)
- added R20: 5.1K, Resistor_SMD:R_0402_1005Metric, F.Cu at (-33.0, -62.5)
- added R21: 10K, all-footprints:RES_ERJ2RKF1002X, F.Cu at (308.0, 127.9)
- added R22: 10K, all-footprints:RES_ERJ2RKF1002X, F.Cu at (308.0, 120.0)
- added R23: 10K, all-footprints:RES_ERJ2RKF1002X, F.Cu at (308.0, 122.0)
- added R24: 10K, all-footprints:RES_ERJ2RKF1002X, F.Cu at (308.0, 126.0)
- added R25: 10K, all-footprints:RES_ERJ2RKF1002X, F.Cu at (325.5, 122.0)
- added R26: 10K, all-footprints:RES_ERJ2RKF1002X, F.Cu at (325.5, 126.0)
- added R29: 220, Resistor_SMD:R_0402_1005Metric, F.Cu at (235.5, 201.5)
- added R3: 5.1K, Resistor_SMD:R_0402_1005Metric, F.Cu at (300.0, 180.0)
- added R30: 220, Resistor_SMD:R_0402_1005Metric, F.Cu at (235.5, 203.0)
- added R31: 10K, all-footprints:RES_ERJ2RKF1002X, F.Cu at (330.0, 120.0)
- added R32: 10K, all-footprints:RES_ERJ2RKF1002X, F.Cu at (334.0, 120.0)
- added R4: 5.1K, Resistor_SMD:R_0402_1005Metric, F.Cu at (305.0, 180.0)
- added R5: 5.1K, Resistor_SMD:R_0402_1005Metric, F.Cu at (-41.7, -68.4)
- added R6: 5.1K, Resistor_SMD:R_0402_1005Metric, F.Cu at (-41.7, -66.5)
- added R7: 5.1K, Resistor_SMD:R_0402_1005Metric, F.Cu at (-41.7, -64.5)
- added R8: 5.1K, Resistor_SMD:R_0402_1005Metric, F.Cu at (-41.7, -62.5)
- added R9: 5.1K, Resistor_SMD:R_0402_1005Metric, F.Cu at (-38.8, -68.4)
- added SW0: OS102011MS2QN1, all-footprints:SPDT_OS102011_CNK, F.Cu at (321.5, 122.0)
- added SW1: OS102011MS2QN1, all-footprints:SPDT_OS102011_CNK, F.Cu at (312.5, 121.9)
- added SW2: OS102011MS2QN1, all-footprints:SPDT_OS102011_CNK, F.Cu at (303.5, 121.9)
- added SW5: OS102011MS2QN1, all-footprints:SPDT_OS102011_CNK, F.Cu at (329.9, 124.5)
- added U1: max4999etj+, all-footprints:21-0140_T3255&plus_4_MXM-M, F.Cu at (277.2, 187.5)
- added U2: FT232HPQ-TRAY, all-footprints:QFN-56_FT232HPQ_FTD, F.Cu at (229.0, 203.0)
- added U3: DG408DJZ, all-footprints:PDIP16_E16.3_REN, F.Cu at (199.9, 279.9)
- added U5: DG408DJZ, all-footprints:PDIP16_E16.3_REN, F.Cu at (299.4, 280.3)
- added Y1: 12MHz, Crystal:Crystal_SMD_2520-4Pin_2.5x2.0mm, F.Cu at (226.9, 210.2)
- moved U4 224.3 mm to (329.0, 111.1), turned to 180 degrees

Commit message: Updating connections to USB output connectors, prepped subsystems for board layout.
Parts:
- moved R13 345.5 mm to (115.4, 242.1)
- moved R14 345.5 mm to (115.4, 244.1)
- moved R19 328.5 mm to (115.4, 228.6)
- moved R20 328.1 mm to (115.4, 230.1)
- moved R17 319.2 mm to (115.4, 214.1)
- moved R18 319.2 mm to (115.4, 216.1)
- moved R15 304.4 mm to (115.4, 199.6)
- moved R16 304.4 mm to (115.4, 201.6)
- moved R11 294.1 mm to (115.6, 185.9)
- moved R12 294.1 mm to (115.6, 187.9)
- moved J8 286.9 mm to (109.4, 229.1), turned to -90 degrees
- moved R10 285.6 mm to (115.8, 173.6)
- moved R9 285.6 mm to (115.8, 171.7)
- moved J7 282.9 mm to (109.5, 215.0), turned to -90 degrees
- moved J6 278.6 mm to (109.5, 200.5), turned to -90 degrees
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Connections:
- J2 pad A12: Net-(J2-GND-PadA1) -> DE9_0_GND
- J2 pad A9: Net-(J2-VBUS-PadA4) -> V_BUS
- J2 pad B12: Net-(J2-GND-PadA1) -> DE9_0_GND
- J2 pad B9: Net-(J2-VBUS-PadA4) -> V_BUS
- J2 pad S1: unconnected-(J2-SHIELD-PadS1) -> DE9_0_GND
- J3 pad A12: Net-(J3-GND-PadA1) -> DE9_0_GND
- J3 pad A9: Net-(J3-VBUS-PadA4) -> V_BUS
- J3 pad B12: Net-(J3-GND-PadA1) -> DE9_0_GND
- J3 pad B9: Net-(J3-VBUS-PadA4) -> V_BUS
- J3 pad S1: unconnected-(J3-SHIELD-PadS1) -> DE9_0_GND
- J4 pad A12: Net-(J4-GND-PadA1) -> DE9_0_GND
- J4 pad A9: Net-(J4-VBUS-PadA4) -> V_BUS
- J4 pad B12: Net-(J4-GND-PadA1) -> DE9_0_GND
- J4 pad B9: Net-(J4-VBUS-PadA4) -> V_BUS
- J4 pad S1: unconnected-(J4-SHIELD-PadS1) -> DE9_0_GND
- J5 pad A12: Net-(J5-GND-PadA1) -> DE9_0_GND
- J5 pad A9: Net-(J5-VBUS-PadA4) -> V_BUS
- J5 pad B12: Net-(J5-GND-PadA1) -> DE9_0_GND
- J5 pad B9: Net-(J5-VBUS-PadA4) -> V_BUS
- J5 pad S1: unconnected-(J5-SHIELD-PadS1) -> DE9_0_GND
- J6 pad A12: Net-(J6-GND-PadA1) -> DE9_0_GND
- J6 pad A9: Net-(J6-VBUS-PadA4) -> V_BUS
- J6 pad B12: Net-(J6-GND-PadA1) -> DE9_0_GND
- J6 pad B9: Net-(J6-VBUS-PadA4) -> V_BUS
- J6 pad S1: unconnected-(J6-SHIELD-PadS1) -> DE9_0_GND
- J7 pad A12: Net-(J7-GND-PadA1) -> DE9_0_GND
- J7 pad A9: Net-(J7-VBUS-PadA4) -> V_BUS
- J7 pad B12: Net-(J7-GND-PadA1) -> DE9_0_GND
- J7 pad B9: Net-(J7-VBUS-PadA4) -> V_BUS
- J7 pad S1: unconnected-(J7-SHIELD-PadS1) -> DE9_0_GND
- J8 pad A12: Net-(J8-GND-PadA1) -> DE9_0_GND
- J8 pad A9: Net-(J8-VBUS-PadA4) -> V_BUS
- J8 pad B12: Net-(J8-GND-PadA1) -> DE9_0_GND
- J8 pad B9: Net-(J8-VBUS-PadA4) -> V_BUS
- J8 pad S1: unconnected-(J8-SHIELD-PadS1) -> DE9_0_GND
- J9 pad A12: Net-(J9-GND-PadA1) -> DE9_0_GND
- J9 pad A9: Net-(J9-VBUS-PadA4) -> V_BUS
- J9 pad B12: Net-(J9-GND-PadA1) -> DE9_0_GND
- J9 pad B9: Net-(J9-VBUS-PadA4) -> V_BUS
- J9 pad S1: unconnected-(J9-SHIELD-PadS1) -> DE9_0_GND

Commit message: Man I have no idea how to layout a board
Parts:
- moved J10 203.8 mm to (361.1, 128.8), turned to 90 degrees
- moved J11 171.8 mm to (361.1, 163.3), turned to 90 degrees
- moved J12 149.2 mm to (361.1, 197.8), turned to 90 degrees
- moved J18 142.9 mm to (246.5, 253.4)
- moved J15 142.9 mm to (348.0, 253.4)
- moved J16 142.9 mm to (314.1, 253.5)
- moved J17 142.9 mm to (280.4, 253.4)
- moved J13 140.6 mm to (361.1, 231.8), turned to 90 degrees
- moved U3 125.1 mm to (303.4, 209.7)
- moved J8 122.7 mm to (231.5, 217.1)
- moved J9 122.7 mm to (231.5, 231.1)
- moved J3 122.7 mm to (231.7, 146.3)
- moved J4 122.7 mm to (231.7, 160.4)
- moved J5 122.7 mm to (231.7, 174.6)
- moved J6 122.7 mm to (231.6, 188.5)
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Routing:
- net DE9_0_GND: track 0.00 -> 113.6 mm
- net Net-(J2-CC1): track 0.00 -> 2.66 mm
- net Net-(J2-CC2): track 0.00 -> 2.66 mm
Other:
- copper layers 2 -> 4
